File: qspibuddy.kicad_pcb (KiCad board)
At the start: 4 copper layers, 65 x 56.5 mm, 51 parts, among them J1 RPi_GPIO, J2 DUT, J3 General Purpose Outputs, J4 UART, J5 Power Outputs, J6 Conn_01x08, J7 Conn_01x08, J8 Conn_01x08, J9 Conn_01x08, Q1 2N7002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

Commit message: routed
Parts:
- removed D1, D3: Red, LED_SMD:LED_0805_2012Metric
- removed D2, D4: Green, LED_SMD:LED_0805_2012Metric
- removed R11, R12, R13, R14: 10k, Resistor_SMD:R_0402_1005Metric
- added R15: 10k, Resistor_SMD:R_0402_1005Metric, F.Cu at (88.7, 54.2)
- added R16: 10k, Resistor_SMD:R_0402_1005Metric, F.Cu at (94.7, 54.2)
- added R17: 10k, Resistor_SMD:R_0402_1005Metric, F.Cu at (67.8, 54.8)
- moved R6 25.0 mm to (64.3, 54.4)
- moved R4 21.6 mm to (70.8, 53.6)
- moved R1 20.7 mm to (96.2, 54.8), turned to -90 degrees
- moved R3 10.9 mm to (69.4, 31.6), turned to -90 degrees
- moved R2 8.30 mm to (64.8, 31.2)
- moved C6 5.33 mm to (101.4, 75.5), turned to -90 degrees
- moved C3 5.27 mm to (76.8, 75.5), turned to -90 degrees
- moved Q1 3.06 mm to (53.6, 38.6)
- moved R7 3.06 mm to (54.6, 31.9)
- moved Q2 3.06 mm to (53.6, 34.2)
- moved R10 3.06 mm to (52.6, 31.9)
- moved R8 3.06 mm to (54.5, 36.4)
- moved R9 3.06 mm to (52.6, 36.4)
- moved R5 2.42 mm to (91.6, 54.1)
- moved U11 2.24 mm to (94.3, 51.0)
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Connections:
- R4 pad 2: /PI_HOLD -> /PI_HOLD_A
- R5 pad 2: /PI_RESET -> /PI_RESET_B
- R6 pad 2: /PI_WP -> /PI_WP_A
- U1 pad 3: /PI_HOLD -> /PI_HOLD_A
- U1 pad 6: /PI_RESET -> /PI_RESET_A
- U3 pad 3: /PI_WP -> /PI_WP_A
- U4 pad 3: /PI_HOLD -> /PI_HOLD_B
- U4 pad 6: /PI_RESET -> /PI_RESET_B
- U5 pad 3: /PI_WP -> /PI_WP_B
Routing:
- net +5V: track 0.00 -> 95.5 mm, vias 0 -> 3
- net /PI_CS: track 0.00 -> 84.4 mm, vias 0 -> 4
- net /PI_DO: track 0.00 -> 79.6 mm, vias 0 -> 6
- net /PI_SCK: track 0.00 -> 77.7 mm, vias 0 -> 3
- net /DUT_DO: track 0.00 -> 67.2 mm, vias 0 -> 6
- net /DUT_HOLD: track 0.00 -> 67.0 mm
- net /DUT_CS: track 0.00 -> 65.3 mm, vias 0 -> 6
- net /DUT_WP: track 0.00 -> 65.1 mm, vias 0 -> 4
- net /PI_DI: track 0.00 -> 63.7 mm, vias 0 -> 4
- net /DUT_RESET: track 0.00 -> 62.8 mm, vias 0 -> 2
- net /PI_POWER_GATE: track 0.00 -> 60.0 mm, vias 0 -> 3
- net /!EN_FLASH_B: track 0.00 -> 57.6 mm, vias 0 -> 6
- net /SEL_FLASH_B: track 0.00 -> 57.5 mm, vias 0 -> 4
- net /DUT_VCC: track 0.00 -> 53.9 mm, vias 0 -> 7
- net GND: track 3.02 -> 55.8 mm, vias 2 -> 38
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- added copper zone on In1.Cu, net +3.3V
- added copper zone on In2.Cu, net /SUPPLY_FLASH_A
- added copper zone on In2.Cu, net /SUPPLY_FLASH_B
Other:
- board text added: "1"
- board text added: "FIXME: Pin labels on Power Outputs"
- board text added: "Flash A"
- board text added: "Flash B"
- board text added: "GND"
- board text added: "GP1"
- board text added: "GP2"
- board text added: "QSPIBuddy"
- board text added: "RXD"
- board text added: "TXD"
- board text added: "kittenlabs.de - RevA"
