File: qspibuddy.kicad_sch (KiCad schematic)
At the start: 51 parts, among them J1 RPi_GPIO, J2 DUT, J3 General Purpose Outputs, J4 UART, J5 Power Outputs, J6 Conn_01x08, J7 Conn_01x08, J8 Conn_01x08, J9 Conn_01x08, Q1 2N7002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

Commit message: routed
Parts:
- removed D1, D3: Red, LED_SMD:LED_0805_2012Metric, symbol Device:LED
- removed D2, D4: Green, LED_SMD:LED_0805_2012Metric, symbol Device:LED
- removed R11, R12, R13, R14: 10k, Resistor_SMD:R_0402_1005Metric, symbol Device:R
- added R15, R16, R17: 10k, Resistor_SMD:R_0402_1005Metric, symbol Device:R
Connections:
- net +3.3V: now also R15.1, R16.1, R17.1
- net PI_HOLD renamed PI_HOLD_A
- net PI_HOLD_A: no longer U4.3 (S1B)
- net PI_RESET renamed PI_RESET_B
- net PI_RESET_B: no longer U1.6 (S2B)
- net PI_WP renamed PI_WP_A
- net PI_WP_A: no longer U5.3 (S1B)
- new net PI_HOLD_B: R16.2, U4.3 (S1B)
- new net PI_RESET_A: R17.2, U1.6 (S2B)
- new net PI_WP_B: R15.2, U5.3 (S1B)
Other:
- moved on the sheet: R5, R6
